File: _autosave-System In Package.sch (KiCad schematic (older format))
At the start: 11 parts, among them U3 OSD3358-512M-BSM

Commit message: Progress
Parts:
- added Q2: MMBT3906, Package_TO_SOT_SMD:SOT-23, symbol Transistor_BJT:MMBT3906
- added R6, R7, R8: R, Resistor_SMD:R_0603_1608Metric, symbol Device:R
- added U5: TLVH431, Package_TO_SOT_SMD:SOT-23, symbol Reference_Voltage:TL431DBZ
Connections:
- net VDD_3V3B: now also Q2.2 (E), R6.1, R8.2
- net VDD_RTC: now also Q2.3 (C), R7.1, U5.3 (A)
- new net: R6.2, R7.2, U5.2 (REF)
- new net: Q2.1 (B), R8.1, U5.1 (K)
Other:
- note added: "Power down - Clamping circuit"
Changed lines of the file:
@@
 $Descr A3 16535 11693
 encoding utf-8
-Sheet 4 4
+Sheet 4 5
 Title ""
 Date ""
@@
 $EndComp
 NoConn ~ 1750 4150
-$Comp
-L PocketBeagle:VDD_RTC #SUPPLY?
-U 1 1 5F711F3F
-P 2000 9850
-F 0 "#SUPPLY?" H 2000 9850 45  0001 L BNN
-F 1 "VDD_RTC" H 2000 10020 45  0000 C CNN
-F 2 "" H 2000 9850 60  0001 C CNN
-F 3 "" H 2000 9850 60  0001 C CNN
-	1    2000 9850
+Wire Notes Line
+	2950 8900 1500 8900
+Text Notes 1500 8850 0    50   ~ 0
+Power down - Clamping circuit
+$Comp
+L PocketBeagle:VDD_3V3B #SUPPLY013
+U 1 1 5F72F7D6
+P 1650 9100
+F 0 "#SUPPLY013" H 1650 9100 45  0001 L BNN
+F 1 "VDD_3V3B" H 1900 9150 45  0000 C CNN
+F 2 "" H 1650 9100 60  0001 C CNN
+F 3 "" H 1650 9100 60  0001 C CNN
+	1    1650 9100
+	1    0    0    -1
+$EndComp
+$Comp
+L Device:R R6
+U 1 1 5F72FA32
+P 1850 9350
+F 0 "R6" H 1920 9396 50  0000 L CNN
+F 1 "R" H 1920 9305 50  0000 L CNN
+F 2 "Resistor_SMD:R_0603_1608Metric" V 1780 9350 50  0001 C CNN
+F 3 "~" H 1850 9350 50  0001 C CNN
+	1    1850 9350
+	1    0    0    -1
+$EndComp
+$Comp
+L Device:R R8
+U 1 1 5F72FE35
+P 2150 9350
+F 0 "R8" H 2080 9304 50  0000 R CNN
+F 1 "R" H 2080 9395 50  0000 R CNN
+F 2 "Resistor_SMD:R_0603_1608Metric" V 2080 9350 50  0001 C CNN
+F 3 "~" H 2150 9350 50  0001 C CNN
+	1    2150 9350
 	-1   0    0    1
 $EndComp
+$Comp
+L Device:R R7
+U 1 1 5F737494
+P 1850 10150
+F 0 "R7" H 1780 10104 50  0000 R CNN
+F 1 "R" H 1780 10195 50  0000 R CNN
+F 2 "Resistor_SMD:R_0603_1608Metric" V 1780 10150 50  0001 C CNN
+F 3 "~" H 1850 10150 50  0001 C CNN
+	1    1850 10150
+	-1   0    0    1
+$EndComp
+Wire Notes Line
+	1500 10700 2950 10700
+Wire Notes Line
+	1500 8900 1500 10700
+Wire Notes Line
+	2950 8900 2950 10700
+Wire Wire Line
+	1650 9200 1850 9200
+Connection ~ 1850 9200
+Wire Wire Line
+	1850 9200 2150 9200
+Wire Wire Line
+	2150 9200 2650 9200
+Wire Wire Line
+	2650 9200 2650 9550
+Connection ~ 2150 9200
+$Comp
+L Transistor_BJT:MMBT3906 Q2
+U 1 1 5F74A472
+P 2550 9750
+F 0 "Q2" H 2741 9704 50  0000 L CNN
+F 1 "MMBT3906" H 2741 9795 50  0000 L CNN
+F 2 "Package_TO_SOT_SMD:SOT-23" H 2750 9675 50  0001 L CIN
+F 3 "https://www.fairchildsemi.com/datasheets/2N/2N3906.pdf" H 2550 9750 50  0001 L CNN
+	1    2550 9750
+	1    0    0    1
+$EndComp
+$Comp
+L Reference_Voltage:TL431DBZ U5
+U 1 1 5F74FB0B
+P 2350 10100
+F 0 "U5" V 2350 10000 50  0000 R CNN
+F 1 "TLVH431" V 2250 10050 50  0000 R CNN
+F 2 "Package_TO_SOT_SMD:SOT-23" H 2350 9950 50  0001 C CIN
+F 3 "http://www.ti.com/lit/ds/symlink/tl431.pdf" H 2350 10100 50  0001 C CIN
+	1    2350 10100
+	0    -1   -1   0
+$EndComp
+Wire Wire Line
+	2200 10100 2200 9750
+Wire Wire Line
+	1850 9750 1850 10000
+Wire Wire Line
+	1850 9500 1850 9750
+Connection ~ 1850 9750
+Wire Wire Line
+	1850 9750 2200 9750
+Wire Wire Line
+	2150 9500 2350 9500
+Wire Wire Line
+	2200 10100 2250 10100
+Wire Wire Line
+	2350 10200 2350 10350
+Wire Wire Line
+	2350 10350 1850 10350
+Wire Wire Line
+	1850 10350 1850 10300
+Wire Wire Line
+	1850 10350 1650 10350
+Wire Wire Line
+	1650 10350 1650 10150
+Connection ~ 1850 10350
+Wire Wire Line
+	2650 9950 2650 10350
+Wire Wire Line
+	2650 10350 2350 10350
+Connection ~ 2350 10350
+$Comp
+L PocketBeagle:VDD_RTC #SUPPLY014
+U 1 1 5F779A9D
+P 1650 10050
+F 0 "#SUPPLY014" H 1650 10050 45  0001 L BNN
+F 1 "VDD_RTC" H 1700 10250 45  0000 C CNN
+F 2 "" H 1650 10050 60  0001 C CNN
+F 3 "" H 1650 10050 60  0001 C CNN
+	1    1650 10050
+	1    0    0    -1
+$EndComp
+Wire Wire Line
+	2350 9500 2350 9750
+Connection ~ 2350 9750
+Wire Wire Line
+	2350 9750 2350 10000
 $EndSCHEMATC
