File: Peripherals.sch (KiCad schematic (older format))
At the start: 1 part, among them J2 Peripheral Header

Commit message: Progress
Connections:
- net labels removed: I2C0_SDA, I2C_SCL
Changed lines of the file:
@@
 	2600 1350 2300 1350
-Wire Wire Line
-	2600 1450 2300 1450
 Wire Wire Line
 	2600 1550 2300 1550
@@
 Wire Wire Line
 	1750 1950 2600 1950
-Wire Wire Line
-	4050 1950 4050 1500
-Wire Wire Line
-	3100 1950 4050 1950
 $Comp
 L power:GND #PWR?
@@
 L PocketBeagle:VDD_5V #SUPPLY?
 U 1 1 5FF95332
-P 4050 1400
+P 1950 1150
 AR Path="/5F8143D2/5FF95332" Ref="#SUPPLY?"  Part="1"
 AR Path="/5F0E396B/5FF95332" Ref="#SUPPLY02"  Part="1"
 AR Path="/5F55F329/5FF95332" Ref="#SUPPLY?"  Part="1"
-F 0 "#SUPPLY02" H 4050 1400 45  0001 L BNN
-F 1 "VDD_5V" H 4050 1570 45  0000 C CNN
-F 2 "" H 4050 1400 60  0001 C CNN
-F 3 "" H 4050 1400 60  0001 C CNN
-	1    4050 1400
+F 0 "#SUPPLY02" H 1950 1150 45  0001 L BNN
+F 1 "VDD_5V" H 1950 1320 45  0000 C CNN
+F 2 "" H 1950 1150 60  0001 C CNN
+F 3 "" H 1950 1150 60  0001 C CNN
+	1    1950 1150
 	1    0    0    -1
 $EndComp
+Text HLabel 3400 1750 2    50   Input ~ 0
+UART0_RX
+Text HLabel 3400 1850 2    50   Output ~ 0
+UART0_TX
+Text HLabel 2300 1850 0    50   Input ~ 0
+ANGL0
+Text HLabel 3400 1950 2    50   Input ~ 0
+MBUS_RST
+Text HLabel 3400 1350 2    50   Input ~ 0
+SPI0_CS0
+Text HLabel 3400 1450 2    50   Input ~ 0
+SPI0_SCLK
 Text HLabel 3400 1550 2    50   Input ~ 0
-UART0_RX
-Text HLabel 3400 1650 2    50   Output ~ 0
-UART0_TX
-Text HLabel 2300 1350 0    50   Input ~ 0
-ANGL0
-Text HLabel 2300 1450 0    50   Input ~ 0
-MBUS_RST
-Text HLabel 2300 1550 0    50   Input ~ 0
-SPI0_CS0
+SPI0_D0
+Text HLabel 3400 1650 2    50   Input ~ 0
+SPI0_D1
+Wire Wire Line
+	1950 1250 1950 1450
+Wire Wire Line
+	1950 1450 2600 1450
+Wire Wire Line
+	3400 1950 3100 1950
 Text HLabel 2300 1650 0    50   Input ~ 0
-SPI0_SCLK
+MBUS_INT
 Text HLabel 2300 1750 0    50   Input ~ 0
-SPI0_D0
-Text HLabel 2300 1850 0    50   Input ~ 0
-SPI0_D1
-Text HLabel 3400 1350 2    50   Input ~ 0
 ECAP_PWM0
-Text HLabel 3400 1450 2    50   Input ~ 0
-MBUS_INT
-Text HLabel 3400 1750 2    50   Input ~ 0
-I2C_SCL
-Text HLabel 3400 1850 2    50   Input ~ 0
-I2C0_SDA
 $EndSCHEMATC

Commit message: Progress - No custom peripheral
Changed lines of the file:
@@
 Text HLabel 3400 1350 2    50   Input ~ 0
 SPI0_CS0
+Text HLabel 3400 1550 2    50   Input ~ 0
+SPI0_SCLK
 Text HLabel 3400 1450 2    50   Input ~ 0
-SPI0_SCLK
-Text HLabel 3400 1550 2    50   Input ~ 0
+SPI0_D1
+Text HLabel 3400 1650 2    50   Input ~ 0
 SPI0_D0
-Text HLabel 3400 1650 2    50   Input ~ 0
-SPI0_D1
 Wire Wire Line
 	1950 1250 1950 1450

Commit message: WIP - Docs & Gerbers (no custom peripheric yet)
Parts:
- added D2, D3, D4, D5: LED, LED_SMD:LED_0201_0603Metric, symbol Device:LED
- added R13, R14, R15, R16: 1.5K, Resistor_SMD:R_0603_1608Metric, symbol Device:R
Connections:
- net labels added: GPIO_A5, GPIO_A6, GPIO_A7, GPIO_A8
- wire segments 18 -> 39
Changed lines of the file:
@@
 Text HLabel 2300 1750 0    50   Input ~ 0
 ECAP_PWM0
+$Comp
+L Device:LED D?
+U 1 1 5F44F8D8
+P 3200 3550
+AR Path="/5F0E3947/5F44F8D8" Ref="D?"  Part="1"
+AR Path="/5F0E396B/5F44F8D8" Ref="D5"  Part="1"
+F 0 "D5" H 3300 3450 50  0000 C CNN
+F 1 "LED" H 3200 3650 50  0000 C CNN
+F 2 "LED_SMD:LED_0201_0603Metric" H 3200 3550 50  0001 C CNN
+F 3 "~" H 3200 3550 50  0001 C CNN
+	1    3200 3550
+	0    -1   -1   0
+$EndComp
+$Comp
+L Device:LED D?
+U 1 1 5F44F8DE
+P 2950 3550
+AR Path="/5F0E3947/5F44F8DE" Ref="D?"  Part="1"
+AR Path="/5F0E396B/5F44F8DE" Ref="D4"  Part="1"
+F 0 "D4" H 3100 3500 50  0000 C CNN
+F 1 "LED" H 2950 3650 50  0000 C CNN
+F 2 "LED_SMD:LED_0201_0603Metric" H 2950 3550 50  0001 C CNN
+F 3 "~" H 2950 3550 50  0001 C CNN
+	1    2950 3550
+	0    -1   -1   0
+$EndComp
+$Comp
+L Device:LED D?
+U 1 1 5F44F8E4
+P 2650 3550
+AR Path="/5F0E3947/5F44F8E4" Ref="D?"  Part="1"
+AR Path="/5F0E396B/5F44F8E4" Ref="D3"  Part="1"
+F 0 "D3" H 2800 3450 50  0000 C CNN
+F 1 "LED" H 2650 3650 50  0000 C CNN
+F 2 "LED_SMD:LED_0201_0603Metric" H 2650 3550 50  0001 C CNN
+F 3 "~" H 2650 3550 50  0001 C CNN
+	1    2650 3550
+	0    -1   -1   0
+$EndComp
+$Comp
+L Device:LED D?
+U 1 1 5F44F8EA
+P 2400 3550
+AR Path="/5F0E3947/5F44F8EA" Ref="D?"  Part="1"
+AR Path="/5F0E396B/5F44F8EA" Ref="D2"  Part="1"
+F 0 "D2" H 2550 3450 50  0000 C CNN
+F 1 "LED" H 2400 3650 50  0000 C CNN
+F 2 "LED_SMD:LED_0201_0603Metric" H 2400 3550 50  0001 C CNN
+F 3 "~" H 2400 3550 50  0001 C CNN
+	1    2400 3550
+	0    -1   -1   0
+$EndComp
+$Comp
+L Device:R R?
+U 1 1 5F44F8F0
+P 2400 3950
+AR Path="/5F0E3947/5F44F8F0" Ref="R?"  Part="1"
+AR Path="/5F0E396B/5F44F8F0" Ref="R13"  Part="1"
+F 0 "R13" H 2470 3996 50  0000 L CNN
+F 1 "1.5K" H 2470 3905 50  0000 L CNN
+F 2 "Resistor_SMD:R_0603_1608Metric" V 2330 3950 50  0001 C CNN
+F 3 "~" H 2400 3950 50  0001 C CNN
+	1    2400 3950
+	1    0    0    -1
+$EndComp
+$Comp
+L Device:R R?
+U 1 1 5F44F8F6
+P 2650 3950
+AR Path="/5F0E3947/5F44F8F6" Ref="R?"  Part="1"
+AR Path="/5F0E396B/5F44F8F6" Ref="R14"  Part="1"
+F 0 "R14" H 2720 3996 50  0000 L CNN
+F 1 "1.5K" H 2720 3905 50  0000 L CNN
+F 2 "Resistor_SMD:R_0603_1608Metric" V 2580 3950 50  0001 C CNN
+F 3 "~" H 2650 3950 50  0001 C CNN
+	1    2650 3950
+	1    0    0    -1
+$EndComp
+$Comp
+L Device:R R?
+U 1 1 5F44F8FC
+P 2950 3950
+AR Path="/5F0E3947/5F44F8FC" Ref="R?"  Part="1"
+AR Path="/5F0E396B/5F44F8FC" Ref="R15"  Part="1"
+F 0 "R15" H 3020 3996 50  0000 L CNN
+F 1 "1.5K" H 3020 3905 50  0000 L CNN
+F 2 "Resistor_SMD:R_0603_1608Metric" V 2880 3950 50  0001 C CNN
+F 3 "~" H 2950 3950 50  0001 C CNN
+	1    2950 3950
+	1    0    0    -1
+$EndComp
+$Comp
+L Device:R R?
+U 1 1 5F44F902
+P 3200 3950
+AR Path="/5F0E3947/5F44F902" Ref="R?"  Part="1"
+AR Path="/5F0E396B/5F44F902" Ref="R16"  Part="1"
+F 0 "R16" H 3270 3996 50  0000 L CNN
+F 1 "1.5K" H 3270 3905 50  0000 L CNN
+F 2 "Resistor_SMD:R_0603_1608Metric" V 3130 3950 50  0001 C CNN
+F 3 "~" H 3200 3950 50  0001 C CNN
+	1    3200 3950
+	1    0    0    -1
+$EndComp
+Wire Wire Line
+	1800 3350 2400 3350
+Wire Wire Line
+	2400 4100 2400 4350
+Wire Wire Line
+	2400 4350 2650 4350
+Wire Wire Line
+	3200 4350 3200 4100
+Wire Wire Line
+	2950 4100 2950 4350
+Connection ~ 2950 4350
+Wire Wire Line
+	2950 4350 3200 4350
+Wire Wire Line
+	2650 4100 2650 4350
+Connection ~ 2650 4350
+Wire Wire Line
+	2650 4350 2800 4350
+Wire Wire Line
+	2650 3400 2650 3250
+Wire Wire Line
+	2650 3250 1800 3250
+Wire Wire Line
+	1800 3150 2950 3150
+Wire Wire Line
+	2950 3150 2950 3400
+Wire Wire Line
+	3200 3400 3200 3050
+Wire Wire Line
+	3200 3050 1800 3050
+Connection ~ 2800 4350
+Wire Wire Line
+	2800 4350 2950 4350
+Wire Wire Line
+	2800 4350 2800 4500
+$Comp
+L power:GND #PWR?
+U 1 1 5F44F91C
+P 2800 4500
+AR Path="/5F0E3947/5F44F91C" Ref="#PWR?"  Part="1"
+AR Path="/5F0E396B/5F44F91C" Ref="#PWR016"  Part="1"
+F 0 "#PWR016" H 2800 4250 50  0001 C CNN
+F 1 "GND" H 2805 4327 50  0000 C CNN
+F 2 "" H 2800 4500 50  0001 C CNN
+F 3 "" H 2800 4500 50  0001 C CNN
+	1    2800 4500
+	1    0    0    -1
+$EndComp
+Text HLabel 1800 3050 0    50   Input ~ 0
+GPIO_A5
+Text HLabel 1800 3150 0    50   Input ~ 0
+GPIO_A6
+Text HLabel 1800 3250 0    50   Input ~ 0
+GPIO_A7
+Text HLabel 1800 3350 0    50   Input ~ 0
+GPIO_A8
+Wire Wire Line
+	2400 3700 2400 3800
+Wire Wire Line
+	2650 3800 2650 3700
+Wire Wire Line
+	2950 3700 2950 3800
+Wire Wire Line
+	3200 3800 3200 3700
+Wire Wire Line
+	2400 3350 2400 3400
 $EndSCHEMATC

Commit message: Custom Peripheral, Gerbers, drills
Parts:
- added C1: 22pF, Capacitor_Tantalum_SMD:CP_EIA-1608-08_AVX-J, symbol Device:C
- added C11: 470nF, Capacitor_Tantalum_SMD:CP_EIA-1608-08_AVX-J, symbol Device:C
- added U8: PCF8883, Package_SO:SOIC-8_3.9x4.9mm_P1.27mm, symbol Sensor_Touch:PCF8883
Connections:
- net labels added: GPIO_CAPTOUCH
- wire segments 39 -> 55
Changed lines of the file:
@@
 Wire Wire Line
 	2400 3350 2400 3400
+$Comp
+L PocketBeagle:VDD_3V3B #SUPPLY0102
+U 1 1 5F2E0A26
+P 5550 1000
+F 0 "#SUPPLY0102" H 5550 1000 45  0001 L BNN
+F 1 "VDD_3V3B" H 5550 1170 45  0000 C CNN
+F 2 "" H 5550 1000 60  0001 C CNN
+F 3 "" H 5550 1000 60  0001 C CNN
+	1    5550 1000
+	1    0    0    -1
+$EndComp
+Wire Wire Line
+	5550 1100 5550 1200
+$Comp
+L power:GND #PWR0101
+U 1 1 5F2E1370
+P 5550 2200
+F 0 "#PWR0101" H 5550 1950 50  0001 C CNN
+F 1 "GND" H 5555 2027 50  0000 C CNN
+F 2 "" H 5550 2200 50  0001 C CNN
+F 3 "" H 5550 2200 50  0001 C CNN
+	1    5550 2200
+	1    0    0    -1
+$EndComp
+$Comp
+L Device:C C1
+U 1 1 5F2E179F
+P 6150 1950
+F 0 "C1" H 6265 1996 50  0000 L CNN
+F 1 "22pF" H 6265 1905 50  0000 L CNN
+F 2 "Capacitor_Tantalum_SMD:CP_EIA-1608-08_AVX-J" H 6188 1800 50  0001 C CNN
+F 3 "~" H 6150 1950 50  0001 C CNN
+	1    6150 1950
+	1    0    0    -1
+$EndComp
+$Comp
+L Device:C C11
+U 1 1 5F2E1CDC
+P 6600 1950
+F 0 "C11" H 6715 1996 50  0000 L CNN
+F 1 "470nF" H 6715 1905 50  0000 L CNN
+F 2 "Capacitor_Tantalum_SMD:CP_EIA-1608-08_AVX-J" H 6638 1800 50  0001 C CNN
+F 3 "~" H 6600 1950 50  0001 C CNN
+	1    6600 1950
+	1    0    0    -1
+$EndComp
+Wire Wire Line
+	5950 1500 6400 1500
+Wire Wire Line
+	5950 1800 6150 1800
+Wire Wire Line
+	6150 2100 5550 2100
+Wire Wire Line
+	5550 2000 5550 2100
+Connection ~ 5550 2100
+Wire Wire Line
+	5550 2100 5550 2200
+Wire Wire Line
+	6600 2100 6150 2100
+Connection ~ 6150 2100
+Wire Wire Line
+	5950 1700 6600 1700
+Wire Wire Line
+	6600 1700 6600 1800
+Wire Wire Line
+	5450 700  5950 700
+Wire Wire Line
+	5950 700  5950 1400
+Wire Wire Line
+	5450 700  5450 1200
+Text HLabel 6400 1500 2    50   Output ~ 0
+GPIO_CAPTOUCH
+$Comp
+L Sensor_Touch:PCF8883 U8
+U 1 1 5F2DE510
+P 5550 1600
+F 0 "U8" H 5100 1700 50  0000 R CNN
+F 1 "PCF8883" H 5100 1800 50  0000 R CNN
+F 2 "Package_SO:SOIC-8_3.9x4.9mm_P1.27mm" H 5450 1250 50  0001 R CNN
+F 3 "http://www.nxp.com/docs/en/data-sheet/PCF8883.pdf" H 5550 1450 50  0001 C CNN
+	1    5550 1600
+	1    0    0    -1
+$EndComp
+Wire Wire Line
+	2300 1350 2300 1000
+Wire Wire Line
+	2300 1000 4500 1000
+Wire Wire Line
+	4500 1000 4500 1600
+Wire Wire Line
+	4500 1600 5150 1600
 $EndSCHEMATC

Commit message: DRC Fixes and more
Parts:
- C1: footprint Capacitor_Tantalum_SMD:CP_EIA-1608-08_AVX-J -> Capacitor_SMD:C_0603_1608Metric
Changed lines of the file:
@@
 F 0 "C1" H 6265 1996 50  0000 L CNN
 F 1 "22pF" H 6265 1905 50  0000 L CNN
-F 2 "Capacitor_Tantalum_SMD:CP_EIA-1608-08_AVX-J" H 6188 1800 50  0001 C CNN
+F 2 "Capacitor_SMD:C_0603_1608Metric" H 6188 1800 50  0001 C CNN
 F 3 "~" H 6150 1950 50  0001 C CNN
 	1    6150 1950
