File: Power Suply.sch (KiCad schematic (older format))
At the start: 7 parts, among them U1 LM2576HVS-5, U2 LM117_TO3

Commit message: Progress
Parts:
- renumbered C1 to C5, C3 to C6, C2 to C7, U2 to U3, U1 to U4
Connections:
- net in_pwr_supply renamed IN_PWR_SUPPLY
Other:
- note added: "O: 3V"
- note added: "O: 5V 1 A"
- moved on the sheet: C5, C6, C7, D1, L1, U3, U4
