File: pcbproyecto.sch (KiCad schematic (older format))
At the start: 6 parts, among them J1 Barrel_Jack_Switch, J2 Conn_02x20_Odd_Even, J3 Micro_SD_Card, J4 USB_A, P1 USB_C_Plug_USB2.0

Commit message: Progress
Parts:
- removed F1: Fuse, Fuse:Fuse_Littelfuse-NANO2-451_453, symbol Device:Fuse
- removed J1: Barrel_Jack_Switch, Connector_BarrelJack:BarrelJack_Horizontal, symbol Connector:Barrel_Jack_Switch
- removed J2: Conn_02x20_Odd_Even, Connector_PinHeader_1.00mm:PinHeader_2x20_P1.00mm_Vertical, symbol Connector_Generic:Conn_02x20_Odd_Even
- removed J3: Micro_SD_Card, Connector_Card:microSD_HC_Hirose_DM3D-SF, symbol Connector:Micro_SD_Card
- removed J4: USB_A, Connector_USB:USB_A_CONNFLY_DS1095-WNR0, symbol Connector:USB_A
- removed P1: USB_C_Plug_USB2.0, Connector_USB:USB_C_Receptacle_Amphenol_12401610E4-2A, symbol Connector:USB_C_Plug_USB2.0
Connections:
- net labels added: USB0_D+, USB0_D-, USB0_ID, USB1_D+, USB1_D-, USB1_VBU
- net labels removed: +5V, GND, UART_RX, UART_TX, USB_DC, VDD_5V
- wire segments 9 -> 63
Other:
- note removed: "Protection"

Commit message: Progress
Parts:
- added FID1, FID2, FID3, FID4: Fiducial, Fiducial:Fiducial_1mm_Mask2mm, symbol Mechanical:Fiducial
Changed lines of the file:
@@
 Text Label 5550 4050 0    50   ~ 0
 USB1_VBU
+Wire Wire Line
+	5300 3350 5650 3350
+Wire Wire Line
+	5650 2900 6500 2900
+Wire Wire Line
+	5650 2900 5650 3350
+$Comp
+L Mechanical:Fiducial FID3
+U 1 1 5FC460AD
+P 2500 7150
+F 0 "FID3" H 2585 7196 50  0000 L CNN
+F 1 "Fiducial" H 2600 7100 50  0000 L CNN
+F 2 "Fiducial:Fiducial_1mm_Mask2mm" H 2500 7150 50  0001 C CNN
+F 3 "~" H 2500 7150 50  0001 C CNN
+	1    2500 7150
+	1    0    0    -1
+$EndComp
+$Comp
+L Mechanical:Fiducial FID4
+U 1 1 5FC4630D
+P 2500 7300
+F 0 "FID4" H 2600 7300 50  0000 L CNN
+F 1 "Fiducial" H 2600 7200 50  0000 L CNN
+F 2 "Fiducial:Fiducial_1mm_Mask2mm" H 2500 7300 50  0001 C CNN
+F 3 "~" H 2500 7300 50  0001 C CNN
+	1    2500 7300
+	1    0    0    -1
+$EndComp
+$Comp
+L Mechanical:Fiducial FID1
+U 1 1 5FC4689D
+P 2350 7150
+F 0 "FID1" H 2100 7200 50  0000 L CNN
+F 1 "Fiducial" H 1950 7100 50  0000 L CNN
+F 2 "Fiducial:Fiducial_1mm_Mask2mm" H 2350 7150 50  0001 C CNN
+F 3 "~" H 2350 7150 50  0001 C CNN
+	1    2350 7150
+	1    0    0    -1
+$EndComp
+$Comp
+L Mechanical:Fiducial FID2
+U 1 1 5FC46A08
+P 2350 7300
+F 0 "FID2" H 2100 7300 50  0000 L CNN
+F 1 "Fiducial" H 1950 7200 50  0000 L CNN
+F 2 "Fiducial:Fiducial_1mm_Mask2mm" H 2350 7300 50  0001 C CNN
+F 3 "~" H 2350 7300 50  0001 C CNN
+	1    2350 7300
+	1    0    0    -1
+$EndComp
+Wire Wire Line
+	6300 1700 6500 1700
 $Sheet
 S 2450 3350 2850 1500
@@
 F15 "MMC0_DAT3" I R 5300 3450 50
 F16 "MMC0_CD" I R 5300 3350 50
+F17 "I2C0_SDA" B L 2450 4550 50
+F18 "I2C0_SCL" B L 2450 4650 50
 $EndSheet
+Text Label 2300 4650 2    50   ~ 0
+I2C1_SCL
+Text Label 2300 4550 2    50   ~ 0
+I2C1_SDA
+Text Label 6300 1800 2    50   ~ 0
+I2C1_SDA
+Text Label 6300 1700 2    50   ~ 0
+I2C1_SCL
 Wire Wire Line
-	5300 3350 5650 3350
+	6300 1800 6500 1800
 Wire Wire Line
-	5650 2900 6500 2900
+	2300 4550 2450 4550
 Wire Wire Line
-	5650 2900 5650 3350
+	2300 4650 2450 4650
 $EndSCHEMATC

Commit message: Progress - No custom peripheral
Changed lines of the file:
@@
 F26 "USB1_VBUS" I L 6500 3850 50
 F27 "MMC0_CD" I L 6500 2900 50
+F28 "PMIC_PGOOD" I L 6500 2300 50
+F29 "WARMRST" I L 6500 2450 50
 $EndSheet
 Wire Wire Line
@@
 F17 "I2C0_SDA" B L 2450 4550 50
 F18 "I2C0_SCL" B L 2450 4650 50
+F19 "PMIC_PGOOD" O L 2450 4200 50
+F20 "WARMRST" O L 2450 4050 50
 $EndSheet
 Text Label 2300 4650 2    50   ~ 0
@@
 Wire Wire Line
 	2300 4650 2450 4650
+Text Label 2300 4200 2    50   ~ 0
+PMIC_PGOOD
+Text Label 2300 4050 2    50   ~ 0
+WARMRST
+Wire Wire Line
+	2300 4050 2450 4050
+Wire Wire Line
+	2300 4200 2450 4200
+Text Label 6350 2450 2    50   ~ 0
+PMIC_PGOOD
+Text Label 6350 2300 2    50   ~ 0
+WARMRST
+Wire Wire Line
+	6350 2300 6500 2300
+Wire Wire Line
+	6350 2450 6500 2450
 $EndSCHEMATC

Commit message: WIP - Docs & Gerbers (no custom peripheric yet)
Connections:
- no-connect marks 0 -> 3
Changed lines of the file:
@@
 F12 "I2C_SCL" I L 6500 5000 50
 F13 "I2C0_SDA" I L 6500 5150 50
+F14 "GPIO_A5" I L 6500 5450 50
+F15 "GPIO_A6" I L 6500 5550 50
+F16 "GPIO_A7" I L 6500 5650 50
+F17 "GPIO_A8" I L 6500 5750 50
 $EndSheet
 $Sheet
@@
 F1 "Protection.sch" 50
 $EndSheet
-Wire Wire Line
-	9250 2600 9550 2600
-Wire Wire Line
-	9250 2500 9650 2500
 $Sheet
 S 2450 1350 2850 1450
@@
 Wire Wire Line
 	2300 3500 2450 3500
-Wire Wire Line
-	9550 4950 9250 4950
-Wire Wire Line
-	9650 5100 9250 5100
-Wire Wire Line
-	9250 1650 10050 1650
-Wire Wire Line
-	10050 5850 9250 5850
-Wire Wire Line
-	9250 5700 9950 5700
-Wire Wire Line
-	9950 1750 9250 1750
-Wire Wire Line
-	9250 1850 9850 1850
-Wire Wire Line
-	9850 5550 9250 5550
-Wire Wire Line
-	9750 1950 9250 1950
-Wire Wire Line
-	9250 5400 9750 5400
 Wire Wire Line
 	6350 4250 6500 4250
@@
 F28 "PMIC_PGOOD" I L 6500 2300 50
 F29 "WARMRST" I L 6500 2450 50
-$EndSheet
-Wire Wire Line
-	9550 2600 9550 4950
-Wire Wire Line
-	9650 2500 9650 5100
-Wire Wire Line
-	9750 1950 9750 5400
-Wire Wire Line
-	9850 1850 9850 5550
-Wire Wire Line
-	9950 1750 9950 5700
-Wire Wire Line
-	10050 1650 10050 5850
+F30 "GPIO_A8" O R 9250 4000 50
+F31 "GPIO_A7" O R 9250 4100 50
+F32 "GPIO_A6" O R 9250 4200 50
+F33 "GPIO_A5" O R 9250 4300 50
+$EndSheet
+Wire Wire Line
+	9850 2600 9850 4950
+Wire Wire Line
+	9950 2500 9950 5100
+Wire Wire Line
+	10050 1950 10050 5400
+Wire Wire Line
+	10150 1850 10150 5550
+Wire Wire Line
+	10250 1750 10250 5700
+Wire Wire Line
+	10350 1650 10350 5850
 Wire Wire Line
 	6200 3950 6200 4150
@@
 Wire Wire Line
 	6350 2450 6500 2450
+Wire Wire Line
+	9250 1650 10350 1650
+Wire Wire Line
+	9250 1750 10250 1750
+Wire Wire Line
+	9250 1850 10150 1850
+Wire Wire Line
+	9250 1950 10050 1950
+Wire Wire Line
+	9250 2500 9950 2500
+Wire Wire Line
+	9250 2600 9850 2600
+Wire Wire Line
+	9250 4950 9850 4950
+Wire Wire Line
+	9250 5100 9950 5100
+Wire Wire Line
+	9250 5400 10050 5400
+Wire Wire Line
+	9250 5550 10150 5550
+Wire Wire Line
+	9250 5700 10250 5700
+Wire Wire Line
+	9250 5850 10350 5850
+Wire Wire Line
+	9250 5250 9300 5250
+NoConn ~ 9300 5250
+Wire Wire Line
+	9250 2300 9500 2300
+Wire Wire Line
+	9250 2400 9500 2400
+NoConn ~ 9500 2300
+NoConn ~ 9500 2400
+Wire Wire Line
+	6250 5450 6500 5450
+Wire Wire Line
+	6500 5550 6250 5550
+Wire Wire Line
+	6250 5650 6500 5650
+Wire Wire Line
+	6250 5750 6500 5750
+Text Label 6250 5450 2    50   ~ 0
+GPIO_A5
+Text Label 6250 5550 2    50   ~ 0
+GPIO_A6
+Text Label 6250 5750 2    50   ~ 0
+GPIO_A8
+Text Label 6250 5650 2    50   ~ 0
+GPIO_A7
+Wire Wire Line
+	9500 4300 9250 4300
+Wire Wire Line
+	9250 4200 9500 4200
+Wire Wire Line
+	9500 4100 9250 4100
+Wire Wire Line
+	9500 4000 9250 4000
+Text Label 9500 4200 0    50   ~ 0
+GPIO_A6
+Text Label 9500 4100 0    50   ~ 0
+GPIO_A7
+Text Label 9500 4000 0    50   ~ 0
+GPIO_A8
+Text Label 9500 4300 0    50   ~ 0
+GPIO_A5
 $EndSCHEMATC

Commit message: Custom Peripheral, Gerbers, drills
Connections:
- no-connect marks 3 -> 5
Changed lines of the file:
@@
 F16 "GPIO_A7" I L 6500 5650 50
 F17 "GPIO_A8" I L 6500 5750 50
+F18 "GPIO_CAPTOUCH" O L 6500 5900 50
 $EndSheet
 $Sheet
@@
 F32 "GPIO_A6" O R 9250 4200 50
 F33 "GPIO_A5" O R 9250 4300 50
+F34 "GPIO_A4" O R 9250 3550 50
 $EndSheet
 Wire Wire Line
@@
 Text Label 9500 4300 0    50   ~ 0
 GPIO_A5
+NoConn ~ 6500 5150
+NoConn ~ 6500 5000
+Wire Wire Line
+	6250 5900 6500 5900
+Text Label 6250 5900 2    50   ~ 0
+GPIO_A4
+Wire Wire Line
+	9500 3550 9250 3550
+Text Label 9500 3550 0    50   ~ 0
+GPIO_A4
 $EndSCHEMATC
