File: pcbproyecto.kicad_pcb (KiCad board)
At the start: 4 copper layers, 75 x 108 mm, 42 parts, among them IC1 SN74LVC1G07DCK, J1 Barrel_Jack_Switch, J3 USB_A, J5 USB_B_Micro, Q1 MMBT3906, Q2 24 MHz, U1 TLVH431, U2 OSD3358-512M-BSM, U3 LM117_TO3, U4 LM2576HVS-5, U5 MICROSD

Commit message: Progress
Parts:
- added C10: 0.1uF, 6.3V, Capacitor_Tantalum_SMD:CP_EIA-1608-08_AVX-J, F.Cu at (78.0, 67.4)
- added FID1: Fiducial, Fiducial:Fiducial_1mm_Mask2mm, F.Cu at (27.2, 21.9)
- added FID2: Fiducial, Fiducial:Fiducial_1mm_Mask2mm, F.Cu at (74.6, 109.8)
- added FID3: Fiducial, Fiducial:Fiducial_1mm_Mask2mm, F.Cu at (74.6, 21.9)
- added FID4: Fiducial, Fiducial:Fiducial_1mm_Mask2mm, F.Cu at (18.0, 109.8)
- added J2: Peripheral Header, Connector_PinHeader_1.00mm:PinHeader_2x08_P1.00mm_Vertical, F.Cu at (32.8, 86.5)
- added J4: EEPROM_GND, Connector_PinHeader_1.00mm:PinHeader_1x01_P1.00mm_Vertical, F.Cu at (76.0, 78.2)
- added J6: EEPROM_WP, Connector_PinHeader_1.00mm:PinHeader_1x01_P1.00mm_Vertical, F.Cu at (79.0, 78.3)
- added R10: 10K, Resistor_SMD:R_0603_1608Metric, F.Cu at (73.5, 67.4)
- added R24: 10K, Resistor_SMD:R_0603_1608Metric, B.Cu at (69.8, 75.7)
- added R25: 10K, Resistor_SMD:R_0603_1608Metric, B.Cu at (69.8, 71.5)
- added R26: 10K, Resistor_SMD:R_0603_1608Metric, B.Cu at (73.5, 71.5)
- added R27: 10K, Resistor_SMD:R_0603_1608Metric, B.Cu at (69.8, 67.2)
- added TP1: TP_PWR_EN, TestPoint:TestPoint_Pad_1.0x1.0mm, F.Cu at (29.6, 25.6)
- added TP2: TP_PWRONSTN, TestPoint:TestPoint_Pad_1.0x1.0mm, F.Cu at (29.6, 29.9)
- added TP3: TP_WAKEUP, TestPoint:TestPoint_Pad_1.0x1.0mm, F.Cu at (32.7, 25.6)
- added TP4: TP_EXTINTN, TestPoint:TestPoint_Pad_1.0x1.0mm, F.Cu at (32.7, 29.9)
- added TP5: TP_I2C_SCL, TestPoint:TestPoint_Pad_1.0x1.0mm, F.Cu at (35.7, 25.6)
- added TP6: TP_I2C_SDA, TestPoint:TestPoint_Pad_1.0x1.0mm, F.Cu at (35.7, 29.9)
- added TP7: TP_VIN_BAT, TestPoint:TestPoint_Pad_1.0x1.0mm, F.Cu at (38.8, 25.6)
- added U6: 24LC32, Package_SO:MSOP-8-1EP_3x3mm_P0.65mm_EP1.68x1.88mm, F.Cu at (73.6, 62.1)
Connections:
- U2 pad A11: (no net) -> /I2C1_SDA
- U2 pad B11: (no net) -> /I2C1_SCL
Routing:
- net /Peripherals/SPI0_D1: track 0.00 -> 41.5 mm, vias 0 -> 1
- net /Peripherals/SPI0_CS0: track 0.00 -> 41.0 mm, vias 0 -> 1
- net /Sistem In Package/AIN51.8V: track 0.00 -> 41.0 mm, vias 0 -> 1
- net /Peripherals/SPI0_D0: track 0.00 -> 40.8 mm, vias 0 -> 1
- net /Peripherals/SPI0_SCLK: track 0.00 -> 39.5 mm, vias 0 -> 1
- net /Sistem In Package/AIN61.8V: track 0.00 -> 37.3 mm, vias 0 -> 1
- net /I2C1_SDA: track 0.00 -> 36.9 mm, vias 0 -> 2
- net /I2C1_SCL: track 0.00 -> 33.0 mm, vias 0 -> 2
- net VDD_5V: track 45.0 -> 77.2 mm
- net VDD_3V3B: track 129.2 -> 161.0 mm
- net /Peripherals/UART0_RX: track 5.21 -> 31.4 mm, vias 0 -> 1
- net /Peripherals/UART0_TX: track 7.20 -> 32.1 mm, vias 0 -> 1
- net Net-(J6-Pad1): track 0.00 -> 21.2 mm, vias 0 -> 2
- net GND: track 131.5 -> 146.4 mm, vias 22 -> 24
- net (no net): track 0.00 -> 4.70 mm
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- added copper zone on F.Cu, net (none)
Other:
- board text added: "Power Circuit"

Commit message: Progress - No custom peripheral
Parts:
- removed C1: 0.1uF , 6.3V, Capacitor_Tantalum_SMD:CP_EIA-1608-08_AVX-J
- added R11: 100K, Resistor_SMD:R_0603_1608Metric, F.Cu at (62.7, 47.8)
- added R12: 100K, Resistor_SMD:R_0603_1608Metric, F.Cu at (66.0, 47.7)
- added RST: PSH_BTN, footprints:MINI_PUSHBUTTON, F.Cu at (74.7, 49.3)
- added U7: TPS3831, Package_SON:Texas_X2SON-4_1x1mm_P0.65mm, F.Cu at (66.0, 43.0)
- IC1: footprint Package_TO_SOT_SMD:SOT-23-5 -> footprints:SC70(TI-DCK)
- moved TP4 85.2 mm to (81.7, 99.5), turned to 90 degrees
- moved TP3 85.1 mm to (81.5, 95.2), turned to 90 degrees
- moved TP2 77.3 mm to (76.6, 91.2), turned to 90 degrees
- moved TP7 53.2 mm to (81.7, 56.9), turned to 90 degrees
- moved TP1 8.74 mm to (38.4, 25.9)
- moved TP6 7.73 mm to (29.1, 25.9)
- moved IC1 3.85 mm to (69.3, 47.5), turned to 180 degrees
- moved TP5 2.47 mm to (33.3, 25.9)
Connections:
- IC1 pad 2: Net-(IC1-Pad2) -> /PMIC_PGOOD
- U2 pad N12: Net-(IC1-Pad2) -> /WARMRST
- U2 pad P11: Net-(IC1-Pad2) -> /WARMRST
- U2 pad R11: Net-(IC1-Pad4) -> /PMIC_PGOOD
Routing:
- net Net-(TP4-Pad1): track 1.27 -> 55.6 mm, vias 0 -> 2
- net Net-(TP1-Pad1): track 1.27 -> 46.4 mm, vias 0 -> 2
- net Net-(TP3-Pad1): track 1.27 -> 43.8 mm, vias 0 -> 2
- net Net-(TP6-Pad1): track 2.13 -> 42.5 mm, vias 1 -> 2
- net Net-(TP5-Pad1): track 2.14 -> 41.6 mm, vias 1 -> 2
- net Net-(TP2-Pad1): track 1.27 -> 35.9 mm, vias 0 -> 2
- net Net-(TP7-Pad1): track 2.54 -> 29.1 mm, vias 0 -> 3
- net Net-(IC1-Pad2): track 25.1 -> 0.00 mm
- net /WARMRST: track 0.00 -> 23.6 mm
- net /PMIC_PGOOD: track 0.00 -> 17.9 mm
- net VDD_RTC: track 86.9 -> 74.4 mm
- net GND: track 146.4 -> 155.5 mm, vias 24 -> 26
- net VDD_3V3B: track 161.0 -> 168.0 mm, vias 3 -> 4
- net Net-(R11-Pad2): track 0.00 -> 5.61 mm
- net (no net): track 4.70 -> 0.33 mm, vias 3 -> 0
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Other:
- rule via_min_size: 0.3048 -> 0.25
- board text added: "3V3"
- board text added: "5V"
- board text added: "GND"
- board text added: "SPI0_CS0"
- board text added: "SPI0_D0"
- board text added: "SPI0_D1"
- board text added: "SPI0_SCLK"
- board text added: "UART0_RX"
- board text added: "UART0_TX"

Commit message: WIP - Docs & Gerbers (no custom peripheric yet)
Parts:
- removed RST: PSH_BTN, footprints:MINI_PUSHBUTTON
- added D2: LED, LED_SMD:LED_0201_0603Metric, F.Cu at (74.4, 38.9)
- added D3: LED, LED_SMD:LED_0201_0603Metric, F.Cu at (74.4, 40.6)
- added D4: LED, LED_SMD:LED_0201_0603Metric, F.Cu at (74.4, 42.9)
- added D5: LED, LED_SMD:LED_0201_0603Metric, F.Cu at (74.5, 45.0)
- added R13: 1.5K, Resistor_SMD:R_0603_1608Metric, F.Cu at (77.5, 38.9)
- added R14: 1.5K, Resistor_SMD:R_0603_1608Metric, F.Cu at (77.5, 40.9)
- added R15: 1.5K, Resistor_SMD:R_0603_1608Metric, F.Cu at (77.5, 42.9)
- added R16: 1.5K, Resistor_SMD:R_0603_1608Metric, F.Cu at (77.5, 45.0)
- added RST1: PSH_BTN, footprints:MINI_PUSHBUTTON, F.Cu at (74.7, 49.5)
- added TP8: TP_SENSE_BAT, TestPoint:TestPoint_Pad_1.0x1.0mm, F.Cu at (70.2, 80.8)
- added TP9: TP_TS_BAT, TestPoint:TestPoint_Pad_1.0x1.0mm, F.Cu at (70.2, 84.0)
Connections:
- U2 pad N6: (no net) -> Net-(TP9-Pad1)
- U2 pad N7: (no net) -> Net-(TP8-Pad1)
- U2 pad P13: (no net) -> /GPIO_A5
- U2 pad P14: (no net) -> /GPIO_A8
- U2 pad R14: (no net) -> /GPIO_A7
- U2 pad T14: (no net) -> /GPIO_A6
Routing:
- net Net-(TP9-Pad1): track 0.00 -> 29.1 mm, vias 0 -> 2
- net /GPIO_A8: track 0.00 -> 27.9 mm, vias 0 -> 2
- net Net-(TP8-Pad1): track 0.00 -> 26.4 mm, vias 0 -> 2
- net /GPIO_A7: track 0.00 -> 25.2 mm, vias 0 -> 2
- net /GPIO_A5: track 0.00 -> 24.0 mm, vias 0 -> 2
- net /GPIO_A6: track 0.00 -> 22.1 mm, vias 0 -> 2
- net GND: track 155.5 -> 163.8 mm
- net Net-(D2-Pad1): track 0.00 -> 2.39 mm
- net Net-(D4-Pad1): track 0.00 -> 2.28 mm
- net Net-(D5-Pad1): track 0.00 -> 2.26 mm
- net Net-(D3-Pad1): track 0.00 -> 2.13 mm
- added copper zone on F.Cu, net Net-(TP2-Pad1)
- added copper zone on F.Cu, net Net-(TP3-Pad1)
- added copper zone on F.Cu, net Net-(TP4-Pad1)
- added copper zone on F.Cu, net Net-(TP7-Pad1)
- added copper zone on F.Cu, net Net-(U2-PadA6)
- added copper zone on Power.Cu, net VDD_3V3B

Commit message: Custom Peripheral, Gerbers, drills
Parts:
- added C1: 22pF, Capacitor_Tantalum_SMD:CP_EIA-1608-08_AVX-J, B.Cu at (68.5, 53.9)
- added C11: 470nF, Capacitor_Tantalum_SMD:CP_EIA-1608-08_AVX-J, B.Cu at (81.2, 59.8)
- added U8: PCF8883, Package_SO:SOIC-8_3.9x4.9mm_P1.27mm, B.Cu at (74.7, 55.1)
Connections:
- J2 pad 1: (no net) -> Net-(J2-Pad1)
- U2 pad A6: (no net) -> Net-(U2-PadA6)
- U2 pad R13: (no net) -> /GPIO_A4
Routing:
- net Net-(J2-Pad1): track 0.00 -> 89.1 mm
- net /GPIO_A4: track 0.00 -> 16.7 mm, vias 0 -> 1
- net Net-(U8-Pad2): track 0.00 -> 14.6 mm
- net GND: track 163.8 -> 176.2 mm
- net Net-(TP7-Pad1): track 29.1 -> 41.2 mm
- net Net-(C11-Pad1): track 0.00 -> 6.31 mm
- net Net-(C1-Pad1): track 0.00 -> 3.70 mm
- net VDD_3V3B: track 168.0 -> 171.2 mm, vias 4 -> 5
