File: pcbproyecto.kicad_pcb (KiCad board)
At the start: 4 copper layers, 75 x 108 mm, 79 parts, among them IC1 SN74LVC1G07DCK, J1 Barrel_Jack_Switch, J2 Peripheral Header, J3 USB_A, J4 EEPROM_GND, J5 USB_B_Micro, J6 EEPROM_WP, Q1 MMBT3906, Q2 24 MHz, U1 TLVH431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

Commit message: Checklist & Small changes, new docs & gerbers
Parts:
- added G***: LOGO, utn:utnlogo100bpi_non_negative_silk, F.Cu at (43.1, 114.8)
- moved J6 5.03 mm to (78.0, 73.4)
- moved TP2 3.40 mm to (80.0, 91.2)
- moved R22 3.20 mm to (73.1, 34.1), turned to 0 degrees
- moved J4 2.72 mm to (78.2, 76.6)
- moved TP4 1.70 mm to (80.0, 99.5)
- moved TP3 1.50 mm to (80.0, 95.2)
- moved TP7 1.12 mm to (80.6, 56.9)
- moved LED1 0.99 mm to (70.3, 37.8), turned to 180 degrees
- turned R11 to 180 degrees
- turned R12 to 180 degrees
- turned R1 to 180 degrees
Routing:
- net Net-(J6-Pad1): track 21.2 -> 15.8 mm
- net Net-(TP2-Pad1): track 35.9 -> 39.3 mm
- net Net-(TP3-Pad1): track 43.8 -> 41.7 mm
- net Net-(TP4-Pad1): track 55.6 -> 54.0 mm
- net Net-(LED1-Pad1): track 2.62 -> 4.14 mm
- net Net-(TP7-Pad1): track 41.2 -> 40.1 mm
- net Net-(R11-Pad2): track 5.61 -> 6.72 mm
- net CGND: track 98.0 -> 99.0 mm
- net /WARMRST: track 23.6 -> 24.4 mm
- net GND: track 176.2 -> 177.0 mm
Other:
- board text added: "1"
- board text added: "2"

Commit message: DRC Fixes and more
Parts:
- removed G***: LOGO, utn:utnlogo100bpi_non_negative_silk
- C1, C10, C2, C3, C4, C8, C9: footprint Capacitor_Tantalum_SMD:CP_EIA-1608-08_AVX-J -> Capacitor_SMD:C_0603_1608Metric
- F1: footprint Fuse:Fuse_Littelfuse-NANO2-451_453 -> footprints:FUSC6125X279N
- R2: value R -> 10K
- R3: value R -> 40K
- R4: value R -> 500
- moved J1 4.65 mm to (32.3, 113.8)
- moved J3 3.08 mm to (25.1, 38.0)
- moved J5 3.00 mm to (16.3, 56.5)
Connections:
- U2 pad A6: Net-(U2-PadA6) -> (no net)
Routing:
- net CGND: track 99.0 -> 4.17 mm, vias 1 -> 0
- net Net-(TP7-Pad1): track 40.1 -> 28.0 mm
- net /Interfaces/IN_PWR_SUPPLY: track 28.0 -> 34.9 mm
- net Net-(TP4-Pad1): track 54.0 -> 50.3 mm
- net /USB0_ID: track 42.0 -> 38.5 mm
- net GND: track 177.0 -> 173.6 mm
- net /USB0_D+: track 42.4 -> 39.1 mm
- net /USB0_D-: track 42.4 -> 39.1 mm
- net /USB1_VBU: track 34.2 -> 37.3 mm
- net USB_DC: track 53.6 -> 56.6 mm
- net /USB1_D+: track 34.7 -> 37.5 mm
- net /USB1_D-: track 34.9 -> 37.4 mm
- net Net-(TP1-Pad1): track 46.4 -> 44.6 mm
- net VDD_3V3A: track 1.27 -> 0.00 mm
- net Net-(TP2-Pad1): track 39.3 -> 40.4 mm
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- added copper zone on F.Cu, net Net-(TP1-Pad1)
- removed copper zone on F.Cu, net (none)
- removed copper zone on F.Cu, net Net-(U2-PadA6)
