File: Interfaces.sch (KiCad schematic (older format))
At the start: 19 parts, among them IC1 SN74LVC1G07DCK, J1 Barrel_Jack_Switch, J3 USB_A, J4 EEPROM_GND, J5 USB_B_Micro, J6 EEPROM_WP, U5 MICROSD, U6 24LC32, U7 TPS3831

Commit message: WIP - Docs & Gerbers (no custom peripheric yet)
Parts:
- renumbered RST to RST1
Changed lines of the file:
@@
 P 2100 6350
 AR Path="/5F0E3947/5FE36935" Ref="PWR?"  Part="1"
-AR Path="/5F8143D2/5FE36935" Ref="RST"  Part="1"
+AR Path="/5F8143D2/5FE36935" Ref="RST1"  Part="1"
 AR Path="/5FC48F0B/5FE36935" Ref="PWR?"  Part="1"
-F 0 "RST" H 2000 6500 45  0000 C CNN
+F 0 "RST1" H 2000 6500 45  0000 C CNN
 F 1 "PSH_BTN" H 2300 6500 45  0000 C CNN
 F 2 "footprints:MINI_PUSHBUTTON" H 2130 6500 20  0001 C CNN

Commit message: DRC Fixes and more
Parts:
- C10, C8, C9: footprint Capacitor_Tantalum_SMD:CP_EIA-1608-08_AVX-J -> Capacitor_SMD:C_0603_1608Metric
Changed lines of the file:
@@
 F 0 "C8" H 8850 2950 50  0000 L CNN
 F 1 "10uF, 10V" H 8550 2750 50  0000 L CNN
-F 2 "Capacitor_Tantalum_SMD:CP_EIA-1608-08_AVX-J" H 8988 2700 50  0001 C CNN
+F 2 "Capacitor_SMD:C_0603_1608Metric" H 8988 2700 50  0001 C CNN
 F 3 "~" H 8950 2850 50  0001 C CNN
 	1    8950 2850
@@
 F 0 "C9" H 9565 2896 50  0000 L CNN
 F 1 "0.1uF 6,3V" H 9565 2805 50  0000 L CNN
-F 2 "Capacitor_Tantalum_SMD:CP_EIA-1608-08_AVX-J" H 9488 2700 50  0001 C CNN
+F 2 "Capacitor_SMD:C_0603_1608Metric" H 9488 2700 50  0001 C CNN
 F 3 "~" H 9450 2850 50  0001 C CNN
 	1    9450 2850
@@
 F 0 "C10" H 3500 4150 50  0000 L CNN
 F 1 "0.1uF, 6.3V" H 3200 3950 50  0000 L CNN
-F 2 "Capacitor_Tantalum_SMD:CP_EIA-1608-08_AVX-J" H 3688 3900 50  0001 C CNN
+F 2 "Capacitor_SMD:C_0603_1608Metric" H 3688 3900 50  0001 C CNN
 F 3 "~" H 3650 4050 50  0001 C CNN
 	1    3650 4050
