File: System In Package.sch (KiCad schematic (older format))
At the start: 2 parts, among them J5 Conn_01x01_Male, U3 OSD3358-512M-BSM

Commit message: Progress
Parts:
- removed J5: Conn_01x01_Male, Connector_PinHeader_1.00mm:PinHeader_1x01_P1.00mm_Vertical, symbol Connector:Conn_01x01_Male
- added LED1: L_PWR, LED_SMD:LED_0603_1608Metric, symbol Device:LED
- added Q?: MMBT3906, Package_TO_SOT_SMD:SOT-23, symbol Transistor_BJT:MMBT3906
- added R1: 1K, Resistor_SMD:R_0603_1608Metric, symbol Device:R
- added R? (x3): R, symbol Device:R
- added RST1: PSH_BTN, footprints:MINI_PUSHBUTTON, symbol PocketBeagle:MINI_PUSHBUTTON
- added TP1: TP_PWR_EN, TestPoint:TestPoint_Pad_1.0x1.0mm, symbol Connector:TestPoint
- added TP2: TP_PWRONSTN, TestPoint:TestPoint_Pad_1.0x1.0mm, symbol Connector:TestPoint
- added TP3: TP_WAKEUP, TestPoint:TestPoint_Pad_1.0x1.0mm, symbol Connector:TestPoint
- added TP4: TP_EXTINTN, TestPoint:TestPoint_Pad_1.0x1.0mm, symbol Connector:TestPoint
- added TP5: TP_I2C_SCL, TestPoint:TestPoint_Pad_1.0x1.0mm, symbol Connector:TestPoint
- added TP6: TP_I2C_SDA, TestPoint:TestPoint_Pad_1.0x1.0mm, symbol Connector:TestPoint
- added TP7: TP_VIN_BAT, TestPoint:TestPoint_Pad_1.0x1.0mm, symbol Connector:TestPoint
- added U?: TLVH431, Package_TO_SOT_SMD:SOT-23, symbol Reference_Voltage:TL431DBZ
Connections:
- net labels added: GND, SYS_5V, VDD_3V3AUX, VDD_3V3B, VDD_RTC
- wire segments 27 -> 116
- no-connect marks 0 -> 1
Other:
- note added: "Power down - Clamping circuit"
- moved on the sheet: U3A, U3B, U3C, U3D, U3E, U3F

Commit message: Progress
Parts:
- removed Q?: MMBT3906, Package_TO_SOT_SMD:SOT-23, symbol Transistor_BJT:MMBT3906
- removed R? (x3): R, symbol Device:R
- removed RST1: PSH_BTN, footprints:MINI_PUSHBUTTON, symbol PocketBeagle:MINI_PUSHBUTTON
- removed U?: TLVH431, Package_TO_SOT_SMD:SOT-23, symbol Reference_Voltage:TL431DBZ
- added C1: 0.1uF , 6.3V, Capacitor_Tantalum_SMD:CP_EIA-1608-08_AVX-J, symbol Device:C
- added C2, C3: 18pF, 50V, Capacitor_Tantalum_SMD:CP_EIA-1608-08_AVX-J, symbol Device:C
- added C4: 0.1uF, 6.3V, Capacitor_Tantalum_SMD:CP_EIA-1608-08_AVX-J, symbol Device:C
- added IC1: SN74LVC1G07DCK, Package_TO_SOT_SMD:SOT-23-5, symbol PocketBeagle:SN74LVC1G07DCK
- added Q2: 24 MHz, Crystal:Crystal_SMD_TXC_7A-2Pin_5x3.2mm, symbol PocketBeagle:CRYSTAL_5X3.2MM
- added R23: 1M , 1%, Resistor_SMD:R_0603_1608Metric, symbol Device:R
- added R24, R25, R26, R27, R5: 10K, Resistor_SMD:R_0603_1608Metric, symbol Device:R
- added R6, R7, R8, R9: 100K, pocketbeagle:RN0804, symbol PocketBeagle:RESISTOR.NETWORK-_4_
- renumbered R1 to R22, U3 to U2
Connections:
- net GND: now also C1.1, IC1.3 (GND), R24.1, R27.1, R5.2, R6.1, R6.2, R6.4, R7.1, R7.2, R7.3, R7.4, R8.2, R8.3, R8.4, R9.1, R9.2, R9.3
- net USB_DC: now also U2.J16 (USB0_VBUS)
- net VDD_3V3B: now also R6.3, R8.1, R9.4
- net VDD_RTC: now also C1.2, IC1.5 (VCC)
- net VDD_1V8: now reaches U2.F10 (SYS_VDD_1P8V)
- net VDD_1V8: now also U2.G10 (SYS_VDD_1P8V), U2.H10 (SYS_VDD_1P8V), U2.H11 (SYS_VDD_1P8V), U2.J10 (SYS_VDD_1P8V), U2.J11 (SYS_VDD_1P8V), U2.K10 (SYS_VDD_1P8V), U2.L10 (SYS_VDD_1P8V)
- net at U2.M16 (RTC_KALDO_ENN): now also R5.1
- net at U2.N12 (PMIC_PGOOD): now also U2.P11 (PWRONRSTN), IC1.2 (A)
- net at U2.R11 (WARMRSTN): now also IC1.4 (Y)
- net PWR_ON: now reaches U2.T11 (PMIC_PB_IN)
- net VREF+: now reaches U2.A7 (SYS_ADC_1P8V)
- net VREF+: now also U2.B7 (VREFP), C4.1
- net AIN01.8V: now reaches U2.A8 (AIN0)
- net VREF-: now reaches U2.A9 (AGND_ADC)
- net VREF-: now also U2.B9 (VREFN), C4.2
- net AIN21.8V: now reaches U2.B6 (AIN2)
- net AIN11.8V: now reaches U2.B8 (AIN1)
- net AIN31.8V: now reaches U2.C6 (AIN3)
- net AIN41.8V: now reaches U2.C7 (AIN4)
- net AIN51.8V: now reaches U2.C8 (AIN5)
- net AIN51.8V: now also R24.2, R25.2
- net AIN61.8V: now reaches U2.C9 (AIN6)
- net AIN61.8V: now also R26.2, R27.2
- net at U2.D6 (PMIC_MUX_OUT): now also U2.D7 (AIN7)
- net USB0_ID: now reaches U2.K14 (USB0_ID)
- net USB0_D+: now reaches U2.K15 (USB0_DP)
- net USB0_D-: now reaches U2.K16 (USB0_DM)
- net USB1_ID: now reaches U2.L14 (USB1_ID)
- net USB1_D+: now reaches U2.L15 (USB1_DP)
- net USB1_D-: now reaches U2.L16 (USB1_DM)
- net USB1_DRVVBUS: now reaches U2.M14 (USB1_DRVVBUS)
- net USB1_VBUS: now reaches U2.M15 (USB1_VBUS)
- net AIN71.8V: now reaches U2.N13 (PMIC_MUX_IN)
- net OSC_GND: now reaches U2.N15 (OSC0_GND)
- net OSC_GND: now also C2.2, C3.2
- net OSC_OUT: now reaches U2.N16 (OSC0_OUT)
- net OSC_OUT: now also C2.1, Q2.1 (P$1), R23.2
- net OSC_IN: now reaches U2.P16 (OSC0_IN)
- net OSC_IN: now also C3.1, Q2.2 (P$2), R23.1
- net I2C2.SCL: now reaches U2.A10 (UART1_RTSN)
- net I2C1.SDA: now reaches U2.A11 (UART1_RXD)
- net SPI0_SCLK: now reaches U2.A13 (SPI0_SCLK)
- net SPI0_CS0: now reaches U2.A14 (SPI0_CS0)
- net MMC0_DAT1: now reaches U2.A15 (MMC0_DAT1)
- net MMC0_DAT0: now reaches U2.A16 (MMC0_DAT0)
- net I2C2.SDA: now reaches U2.B10 (UART1_CTSN)
- net I2C1.SCL: now reaches U2.B11 (UART1_TXD)
- net SPI0_D0: now reaches U2.B13 (SPI0_D0)
- net SPI0_D1: now reaches U2.B14 (SPI0_D1)
- net MMC0_CLK: now reaches U2.B15 (MMC0_CLK)
- net MMC0_CMD: now reaches U2.B16 (MMC0_CMD)
- net SPI1.MIS0: now reaches U2.C12 (UART0_CTSN)
- net SPI1.MOSI: now reaches U2.C13 (UART0_RTSN)
- net MMC0_CD: now reaches U2.C14 (SPI0_CS1)
- net MMC0_DAT3: now reaches U2.C15 (MMC0_DAT3)
- net MMC0_DAT2: now reaches U2.C16 (MMC0_DAT2)
- net LCD_D2_G1: now reaches U2.G1 (LCD_DATA2)
- net LCD_D2_G1: now also R9.6
- net LCD_D1_G2: now reaches U2.G2 (LCD_DATA1)
- net LCD_D1_G2: now also R9.7
- net LCD_D0_G3: now reaches U2.G3 (LCD_DATA0)
- net LCD_D0_G3: now also R9.8
- net LCD_D5_H1: now reaches U2.H1 (LCD_DATA5)
- net LCD_D5_H1: now also R8.7
- net LCD_D4_H2: now reaches U2.H2 (LCD_DATA4)
- net LCD_D4_H2: now also R8.8
- net LCD_D3_H3: now reaches U2.H3 (LCD_DATA3)
- net LCD_D3_H3: now also R9.5
- net LCD_D8_J1: now reaches U2.J1 (LCD_DATA8)
- net LCD_D8_J1: now also R7.8
- net LCD_D7_J2: now reaches U2.J2 (LCD_DATA7)
- net LCD_D7_J2: now also R8.5
- net LCD_D6_J3: now reaches U2.J3 (LCD_DATA6)
- net LCD_D6_J3: now also R8.6
- net LCD_D11_K1: now reaches U2.K1 (LCD_DATA11)
- net LCD_D11_K1: now also R7.5
- net LCD_D10_K2: now reaches U2.K2 (LCD_DATA10)
- net LCD_D10_K2: now also R7.6
- net LCD_D9_K3: now reaches U2.K3 (LCD_DATA9)
- net LCD_D9_K3: now also R7.7
- net LCD_D14_L1: now reaches U2.L1 (LCD_DATA14)
- net LCD_D14_L1: now also R6.6
- net LCD_D13_L2: now reaches U2.L2 (LCD_DATA13)
- net LCD_D13_L2: now also R6.7
- net LCD_D12_L3: now reaches U2.L3 (LCD_DATA12)
- net LCD_D12_L3: now also R6.8
- net LCD_D15_M3: now reaches U2.M3 (LCD_DATA15)
- net LCD_D15_M3: now also R6.5
- new net AIN53.3V: R25.1
- new net AIN63.3V: R26.1
- no-connect marks 1 -> 59
Other:
- note added: "0"
- note added: "1"
- note added: "Boot configuration"
- note added: "Client"
- note added: "HOST"
- note removed: "Power down - Clamping circuit"
- moved on the sheet: U2D

Commit message: Progress - No custom peripheral
Parts:
- removed C1: 0.1uF , 6.3V, Capacitor_Tantalum_SMD:CP_EIA-1608-08_AVX-J, symbol Device:C
- removed IC1: SN74LVC1G07DCK, Package_TO_SOT_SMD:SOT-23-5, symbol PocketBeagle:SN74LVC1G07DCK
Connections:
- net PMIC_PGOOD: now reaches U2.N12 (PMIC_PGOOD), U2.P11 (PWRONRSTN)
- net WARMRST: now reaches U2.R11 (WARMRSTN)
Changed lines of the file:
@@
 $EndComp
 NoConn ~ 1750 4150
-$Comp
-L PocketBeagle:SN74LVC1G07DCK IC1
-U 1 1 5F919AC6
-P 4900 7250
-AR Path="/5F0E3947/5F919AC6" Ref="IC1"  Part="1"
-AR Path="/5FB20BFB/5F919AC6" Ref="IC?"  Part="1"
-AR Path="/5F55F34C/5F919AC6" Ref="IC?"  Part="1"
-F 0 "IC1" H 5000 7400 45  0000 C CNN
-F 1 "SN74LVC1G07DCK" H 5250 7150 45  0000 C CNN
-F 2 "Package_TO_SOT_SMD:SOT-23-5" H 4930 7400 20  0001 C CNN
-F 3 "" H 4900 7250 60  0001 C CNN
-	1    4900 7250
-	1    0    0    -1
-$EndComp
-$Comp
-L power:GND #PWR024
-U 1 1 5F91B3AE
-P 4900 7350
-AR Path="/5F0E3947/5F91B3AE" Ref="#PWR024"  Part="1"
-AR Path="/5FB20BFB/5F91B3AE" Ref="#PWR?"  Part="1"
-AR Path="/5F55F34C/5F91B3AE" Ref="#PWR?"  Part="1"
-F 0 "#PWR024" H 4900 7100 50  0001 C CNN
-F 1 "GND" H 4905 7177 50  0000 C CNN
-F 2 "" H 4900 7350 50  0001 C CNN
-F 3 "" H 4900 7350 50  0001 C CNN
-	1    4900 7350
-	1    0    0    -1
-$EndComp
 Wire Wire Line
 	4550 7150 4550 7250
-Wire Wire Line
-	4700 7250 4550 7250
-Wire Wire Line
-	4550 7650 5100 7650
-Wire Wire Line
-	5100 7650 5100 7250
-Wire Wire Line
-	4900 7000 4900 7150
 $Comp
 L PocketBeagle:VDD_RTC #SUPPLY020
 U 1 1 5F94AFD0
-P 4900 6900
+P 4900 6650
 AR Path="/5F0E3947/5F94AFD0" Ref="#SUPPLY020"  Part="1"
 AR Path="/5FB20BFB/5F94AFD0" Ref="#SUPPLY?"  Part="1"
 AR Path="/5F55F34C/5F94AFD0" Ref="#SUPPLY?"  Part="1"
-F 0 "#SUPPLY020" H 4900 6900 45  0001 L BNN
-F 1 "VDD_RTC" H 4900 7070 45  0000 C CNN
-F 2 "" H 4900 6900 60  0001 C CNN
-F 3 "" H 4900 6900 60  0001 C CNN
-	1    4900 6900
-	1    0    0    -1
-$EndComp
-Wire Wire Line
-	4900 7000 5100 7000
-Connection ~ 4900 7000
-$Comp
-L Device:C C1
-U 1 1 5F96982C
-P 5250 7000
-AR Path="/5F0E3947/5F96982C" Ref="C1"  Part="1"
-AR Path="/5FB20BFB/5F96982C" Ref="C?"  Part="1"
-AR Path="/5F55F34C/5F96982C" Ref="C?"  Part="1"
-F 0 "C1" V 4998 7000 50  0000 C CNN
-F 1 "0.1uF , 6.3V" V 5100 7200 50  0000 C CNN
-F 2 "Capacitor_Tantalum_SMD:CP_EIA-1608-08_AVX-J" H 5288 6850 50  0001 C CNN
-F 3 "~" H 5250 7000 50  0001 C CNN
-	1    5250 7000
-	0    1    1    0
-$EndComp
-$Comp
-L power:GND #PWR026
-U 1 1 5F96A7CF
-P 5400 7000
-AR Path="/5F0E3947/5F96A7CF" Ref="#PWR026"  Part="1"
-AR Path="/5FB20BFB/5F96A7CF" Ref="#PWR?"  Part="1"
-AR Path="/5F55F34C/5F96A7CF" Ref="#PWR?"  Part="1"
-F 0 "#PWR026" H 5400 6750 50  0001 C CNN
-F 1 "GND" V 5405 6872 50  0000 R CNN
-F 2 "" H 5400 7000 50  0001 C CNN
-F 3 "" H 5400 7000 50  0001 C CNN
-	1    5400 7000
-	0    -1   -1   0
+F 0 "#SUPPLY020" H 4900 6650 45  0001 L BNN
+F 1 "VDD_RTC" H 4900 6820 45  0000 C CNN
+F 2 "" H 4900 6650 60  0001 C CNN
+F 3 "" H 4900 6650 60  0001 C CNN
+	1    4900 6650
+	1    0    0    -1
 $EndComp
 Wire Wire Line
@@
 	0    1    1    0
 $EndComp
-Connection ~ 4550 7250
 Wire Wire Line
 	4550 4950 4550 5050
@@
 NoConn ~ 13800 5550
 NoConn ~ 13800 5650
+Text HLabel 4550 7150 2    50   Input ~ 0
+PMIC_PGOOD
+Text HLabel 4550 7650 2    50   Input ~ 0
+WARMRST
 $EndSCHEMATC

Commit message: WIP - Docs & Gerbers (no custom peripheric yet)
Parts:
- added TP8: TP_SENSE_BAT, TestPoint:TestPoint_Pad_1.0x1.0mm, symbol Connector:TestPoint
- added TP9: TP_TS_BAT, TestPoint:TestPoint_Pad_1.0x1.0mm, symbol Connector:TestPoint
Connections:
- net at U2.N6 (PMIC_TS): now also TP9.1
- net at U2.N7 (PMIC_BAT_SENSE): now also TP8.1
- net GPIO_A5: now reaches U2.P13 (GPMC_A5)
- net GPIO_A8: now reaches U2.P14 (GPMC_A8)
- net GPIO_A7: now reaches U2.R14 (GPMC_A7)
- net GPIO_A6: now reaches U2.T14 (GPMC_A6)
- no-connect marks 59 -> 55
Changed lines of the file:
@@
 NoConn ~ 13800 1650
 NoConn ~ 13800 1750
-NoConn ~ 13800 1850
-NoConn ~ 13800 1950
-NoConn ~ 13800 2050
-NoConn ~ 13800 2150
 NoConn ~ 13800 2250
 NoConn ~ 13800 2350
@@
 Text HLabel 4550 7650 2    50   Input ~ 0
 WARMRST
+$Comp
+L Connector:TestPoint TP8
+U 1 1 5F2C20E2
+P 1750 2850
+AR Path="/5F0E3947/5F2C20E2" Ref="TP8"  Part="1"
+AR Path="/5FB20BFB/5F2C20E2" Ref="TP?"  Part="1"
+AR Path="/5F55F34C/5F2C20E2" Ref="TP?"  Part="1"
+F 0 "TP8" V 1850 2850 50  0000 L CNN
+F 1 "TP_SENSE_BAT" V 1750 3100 50  0000 L CNN
+F 2 "TestPoint:TestPoint_Pad_1.0x1.0mm" H 1950 2850 50  0001 C CNN
+F 3 "~" H 1950 2850 50  0001 C CNN
+	1    1750 2850
+	0    -1   -1   0
+$EndComp
+$Comp
+L Connector:TestPoint TP9
+U 1 1 5F2C2C70
+P 1750 2950
+AR Path="/5F0E3947/5F2C2C70" Ref="TP9"  Part="1"
+AR Path="/5FB20BFB/5F2C2C70" Ref="TP?"  Part="1"
+AR Path="/5F55F34C/5F2C2C70" Ref="TP?"  Part="1"
+F 0 "TP9" V 1650 2950 50  0000 L CNN
+F 1 "TP_TS_BAT" V 1750 3200 50  0000 L CNN
+F 2 "TestPoint:TestPoint_Pad_1.0x1.0mm" H 1950 2950 50  0001 C CNN
+F 3 "~" H 1950 2950 50  0001 C CNN
+	1    1750 2950
+	0    -1   -1   0
+$EndComp
+Text HLabel 13900 2150 2    50   Output ~ 0
+GPIO_A8
+Text HLabel 13900 2050 2    50   Output ~ 0
+GPIO_A7
+Text HLabel 13900 1950 2    50   Output ~ 0
+GPIO_A6
+Text HLabel 13900 1850 2    50   Output ~ 0
+GPIO_A5
+Wire Wire Line
+	13800 1850 13900 1850
+Wire Wire Line
+	13800 1950 13900 1950
+Wire Wire Line
+	13800 2050 13900 2050
+Wire Wire Line
+	13800 2150 13900 2150
 $EndSCHEMATC

Commit message: Custom Peripheral, Gerbers, drills
Connections:
- net GPIO_A4: now reaches U2.R13 (GPMC_A4)
- no-connect marks 55 -> 54
Changed lines of the file:
@@
 NoConn ~ 13800 1550
 NoConn ~ 13800 1650
-NoConn ~ 13800 1750
 NoConn ~ 13800 2250
 NoConn ~ 13800 2350
@@
 Wire Wire Line
 	13800 2150 13900 2150
+Text HLabel 13900 1750 2    50   Output ~ 0
+GPIO_A4
+Wire Wire Line
+	13800 1750 13900 1750
 $EndSCHEMATC

Commit message: DRC Fixes and more
Parts:
- C2, C3, C4: footprint Capacitor_Tantalum_SMD:CP_EIA-1608-08_AVX-J -> Capacitor_SMD:C_0603_1608Metric
Changed lines of the file:
@@
 F 0 "C2" V 5400 2250 50  0000 C CNN
 F 1 "18pF, 50V" V 5700 2250 50  0000 C CNN
-F 2 "Capacitor_Tantalum_SMD:CP_EIA-1608-08_AVX-J" H 5588 2100 50  0001 C CNN
+F 2 "Capacitor_SMD:C_0603_1608Metric" H 5588 2100 50  0001 C CNN
 F 3 "~" H 5550 2250 50  0001 C CNN
 	1    5550 2250
@@
 F 0 "C3" V 5450 1650 50  0000 C CNN
 F 1 "18pF, 50V" V 5750 1650 50  0000 C CNN
-F 2 "Capacitor_Tantalum_SMD:CP_EIA-1608-08_AVX-J" H 5638 1500 50  0001 C CNN
+F 2 "Capacitor_SMD:C_0603_1608Metric" H 5638 1500 50  0001 C CNN
 F 3 "~" H 5600 1650 50  0001 C CNN
 	1    5600 1650
@@
 F 0 "C4" H 9615 2546 50  0000 L CNN
 F 1 "0.1uF, 6.3V" H 9615 2455 50  0000 L CNN
-F 2 "Capacitor_Tantalum_SMD:CP_EIA-1608-08_AVX-J" H 9538 2350 50  0001 C CNN
+F 2 "Capacitor_SMD:C_0603_1608Metric" H 9538 2350 50  0001 C CNN
 F 3 "~" H 9500 2500 50  0001 C CNN
 	1    9500 2500
